File: esp8266-bb-mini.sch (KiCad schematic (older format))
At the start: 17 parts, among them J1 Conn_01x02_Male, J2 Conn_01x04_Male, J3 Conn_01x04_Male, J4 Conn_01x04_Male, J5 Conn_01x04_Male, U1 LP38693MP-3.3, U2 ESP-12F

Commit message: sch: add power flags
Signed-off-by: Tillmann Heidsieck <theidsieck@leenox.de>
Changed lines of the file:
@@
 	-1   0    0    1
 $EndComp
+$Comp
+L power:PWR_FLAG #FLG0101
+U 1 1 5FC6F48A
+P 9000 2150
+F 0 "#FLG0101" H 9000 2225 50  0001 C CNN
+F 1 "PWR_FLAG" H 9000 2323 50  0000 C CNN
+F 2 "" H 9000 2150 50  0001 C CNN
+F 3 "~" H 9000 2150 50  0001 C CNN
+	1    9000 2150
+	1    0    0    -1
+$EndComp
+Wire Wire Line
+	8700 2150 9000 2150
+Connection ~ 8700 2150
+$Comp
+L power:PWR_FLAG #FLG0102
+U 1 1 5FC71955
+P 9000 2250
+F 0 "#FLG0102" H 9000 2325 50  0001 C CNN
+F 1 "PWR_FLAG" H 9000 2423 50  0000 C CNN
+F 2 "" H 9000 2250 50  0001 C CNN
+F 3 "~" H 9000 2250 50  0001 C CNN
+	1    9000 2250
+	-1   0    0    1
+$EndComp
+Wire Wire Line
+	9000 2250 8700 2250
+Connection ~ 8700 2250
 $EndSCHEMATC
